File: WiringHarness.kicad_sch (KiCad schematic)
At the start: 39 parts, among them J32 Conn_01x02_Pin, J33 Conn_01x02_Socket, SW1 SW_MEC_5G, SW13 SW_Push, SW14 SW_Push, SW15 SW_Push, SW16 SW_Push, SW17 SW_Push, SW2 SW_MEC_5G, SW24 SW_Push, SW25 SW_Push, SW27 SW_Push, SW28 SW_Push, SW3 SW_MEC_5G, SW30 SW_Push, SW31 SW_Push, SW33 SW_Push

Commit message: changed battery connector
Parts:
- removed U5, U6: (no value), symbol velion:QS9-s
