File: WiringHarness.kicad_sch (KiCad schematic)
At the start: 37 parts, among them J32 Conn_01x02_Pin, J33 Conn_01x02_Socket, SW1 SW_MEC_5G, SW13 SW_Push, SW14 SW_Push, SW15 SW_Push, SW16 SW_Push, SW17 SW_Push, SW2 SW_MEC_5G, SW24 SW_Push, SW25 SW_Push, SW27 SW_Push, SW28 SW_Push, SW3 SW_MEC_5G, SW30 SW_Push, SW31 SW_Push, SW33 SW_Push

Commit message: added measured lenght velion
Other:
- note added: "0.7m"
- note added: "0.9m"
- note added: "1.1m"
- note added: "1.2m"
- note added: "1.4m"
- note added: "1.8m"
- note added: "2m"
Changed lines of the file:
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@@
+		)
+	)
+	(text "1.4m"
+		(exclude_from_sim no)
+		(at 327.152 924.052 0)
+		(effects
+			(font
+				(size 1.27 1.27)
+			)
 		)
 	)
@@
 		)
 	)
+	(text "0.7m"
+		(exclude_from_sim no)
+		(at 352.298 502.92 0)
+		(effects
+			(font
+				(size 1.27 1.27)
+			)
+		)
+	)
 	(text "85 CHF"
 		(exclude_from_sim no)
@@
 		)
 	)
+	(text "0.9m"
+		(exclude_from_sim no)
+		(at 393.446 351.79 0)
+		(effects
+			(font
+				(size 1.27 1.27)
+			)
+		)
+	)
 	(text "left blinker button"
 		(exclude_from_sim no)
@@
 		)
 	)
+	(text "1.4m"
+		(exclude_from_sim no)
+		(at 153.67 849.63 0)
+		(effects
+			(font
+				(size 1.27 1.27)
+			)
+		)
+	)
 	(text "Side light Right"
 		(exclude_from_sim no)
@@
 		)
 	)
+	(text "2m"
+		(exclude_from_sim no)
+		(at 237.998 740.156 0)
+		(effects
+			(font
+				(size 1.27 1.27)
+			)
+		)
+	)
 	(text "right blinker button"
 		(exclude_from_sim no)
@@
 		)
 	)
+	(text "2m"
+		(exclude_from_sim no)
+		(at 210.058 711.2 0)
+		(effects
+			(font
+				(size 1.27 1.27)
+			)
+		)
+	)
 	(text "Regen"
 		(exclude_from_sim no)
@@
 		)
 	)
+	(text "2m"
+		(exclude_from_sim no)
+		(at 155.448 809.244 0)
+		(effects
+			(font
+				(size 1.27 1.27)
+			)
+		)
+	)
 	(text "RIGHT\n"
 		(exclude_from_sim no)
@@
 		)
 	)
+	(text "2m"
+		(exclude_from_sim no)
+		(at 210.312 774.446 0)
+		(effects
+			(font
+				(size 1.27 1.27)
+			)
+		)
+	)
 	(text "Led Position Optionnel Retro"
 		(exclude_from_sim no)
@@
 		)
 	)
+	(text "1.1m"
+		(exclude_from_sim no)
+		(at 358.902 581.66 0)
+		(effects
+			(font
+				(size 1.27 1.27)
+			)
+		)
+	)
 	(text "Z209BG P 00 A0 1000"
 		(exclude_from_sim no)
@@
 		)
 	)
+	(text "1.8m"
+		(exclude_from_sim no)
+		(at 271.018 889.508 0)
+		(effects
+			(font
+				(size 1.27 1.27)
+			)
+		)
+	)
 	(text "Assist A/B quadrature + click Input"
 		(exclude_from_sim no)
@@
 		)
 	)
+	(text "2m"
+		(exclude_from_sim no)
+		(at 353.822 123.444 0)
+		(effects
+			(font
+				(size 1.27 1.27)
+			)
+		)
+	)
 	(text "bonus for speed limiter"
 		(exclude_from_sim no)
@@
 		(exclude_from_sim no)
 		(at 504.444 989.33 0)
+		(effects
+			(font
+				(size 1.27 1.27)
+			)
+		)
+	)
+	(text "2m"
+		(exclude_from_sim no)
+		(at 152.146 822.198 0)
 		(effects
 			(font
@@
 		)
 	)
+	(text "2m"
+		(exclude_from_sim no)
+		(at 360.426 442.468 0)
+		(effects
+			(font
+				(size 1.27 1.27)
+			)
+		)
+	)
 	(text "2 quad input"
 		(exclude_from_sim no)
@@
 		(effects
 			(font
+				(size 1.27 1.27)
+			)
+		)
+	)
+	(text "1.2m"
+		(exclude_from_sim no)
+		(at 368.3 274.32 0)
+		(effects
+			(font
