File: WiringHarness.kicad_sch (KiCad schematic)
At the start: 37 parts, among them J32 Conn_01x02_Pin, J33 Conn_01x02_Socket, SW1 SW_MEC_5G, SW13 SW_Push, SW14 SW_Push, SW15 SW_Push, SW16 SW_Push, SW17 SW_Push, SW2 SW_MEC_5G, SW24 SW_Push, SW25 SW_Push, SW27 SW_Push, SW28 SW_Push, SW3 SW_MEC_5G, SW30 SW_Push, SW31 SW_Push, SW33 SW_Push

Commit message: clean schematic + gitignore
Other:
- note added: "NO FRENCH FIX FOR NEXT WEEK"
- note added: "dont go trough the connector"
Changed lines of the file:
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@@
+		)
+	)
+	(text "dont go trough the connector"
+		(exclude_from_sim no)
+		(at 178.054 281.686 0)
+		(effects
+			(font
+				(size 1.27 1.27)
+			)
+			(justify left)
 		)
 	)
@@
 		)
 	)
+	(text "NO FRENCH\nFIX FOR NEXT WEEK"
+		(exclude_from_sim no)
+		(at 170.18 -98.552 0)
+		(effects
+			(font
+				(size 20 20)
+			)
+			(justify left)
+		)
+	)
